Commit message: add back package:// delimeter

File: urdf/j2s7s300_standalone.urdf (robot description, URDF)
Before this commit: robot j2s7s300, 16 links, 15 joints
Links:
- link j2s7s300_link_1: geometry collision mesh filename=package://kinova_description/meshes/shoulder.dae; visual mesh filename=package://kinova_description/meshes/ring_big.STL
- link j2s7s300_link_2: geometry collision mesh filename=package://kinova_description/meshes/arm_half_1.dae; visual mesh filename=package://kinova_description/meshes/arm_half_1.dae
- link j2s7s300_link_3: geometry collision mesh filename=package://kinova_description/meshes/arm_half_2.dae; visual mesh filename=package://kinova_description/meshes/arm_half_2.dae
- link j2s7s300_link_4: geometry collision mesh filename=package://kinova_description/meshes/forearm.dae; visual mesh filename=package://kinova_description/meshes/forearm.dae
- link j2s7s300_link_5: geometry collision mesh filename=package://kinova_description/meshes/wrist_spherical_1.dae; visual mesh filename=package://kinova_description/meshes/ring_small.STL
- link j2s7s300_link_6: geometry collision mesh filename=package://kinova_description/meshes/wrist_spherical_2.dae; visual mesh filename=package://kinova_description/meshes/ring_small.STL
- link j2s7s300_link_7: geometry collision mesh filename=package://kinova_description/meshes/hand_3finger.dae; visual mesh filename=package://kinova_description/meshes/hand_3finger.dae
- link j2s7s300_link_base: geometry collision mesh filename=package://kinova_description/meshes/base.dae; visual mesh filename=package://kinova_description/meshes/base.dae
- link j2s7s300_link_finger_1: geometry collision mesh filename=package://kinova_description/meshes/finger_proximal.dae; visual mesh filename=package://kinova_description/meshes/finger_proximal.dae
- link j2s7s300_link_finger_2: geometry collision mesh filename=package://kinova_description/meshes/finger_proximal.dae; visual mesh filename=package://kinova_description/meshes/finger_proximal.dae
- link j2s7s300_link_finger_3: geometry collision mesh filename=package://kinova_description/meshes/finger_proximal.dae; visual mesh filename=package://kinova_description/meshes/finger_proximal.dae
