Commit message: add package delimeter back to m1n6s300

File: urdf/m1n6s300_standalone.urdf (robot description, URDF)
Before this commit: robot m1n6s300, 18 links, 17 joints
Links:
- link m1n6s300_link_1: geometry collision mesh filename=package://kinova_description/meshes/shoulder.dae; visual mesh filename=package://kinova_description/meshes/ring_big.STL
- link m1n6s300_link_2: geometry collision mesh filename=package://kinova_description/meshes/arm_mico.dae; visual mesh filename=package://kinova_description/meshes/arm_mico.dae
- link m1n6s300_link_3: geometry collision mesh filename=package://kinova_description/meshes/forearm_mico.dae; visual mesh filename=package://kinova_description/meshes/forearm_mico.dae
- link m1n6s300_link_4: geometry collision mesh filename=package://kinova_description/meshes/wrist.dae; visual mesh filename=package://kinova_description/meshes/ring_small.STL
- link m1n6s300_link_5: geometry collision mesh filename=package://kinova_description/meshes/wrist.dae; visual mesh filename=package://kinova_description/meshes/ring_small.STL
- link m1n6s300_link_6: geometry collision mesh filename=package://kinova_description/meshes/hand_3finger.dae; visual mesh filename=package://kinova_description/meshes/hand_3finger.dae
- link m1n6s300_link_base: geometry collision mesh filename=package://kinova_description/meshes/base.dae; visual mesh filename=package://kinova_description/meshes/base.dae
- link m1n6s300_link_finger_1: geometry collision mesh filename=package://kinova_description/meshes/finger_proximal.dae; visual mesh filename=package://kinova_description/meshes/finger_proximal.dae
- link m1n6s300_link_finger_2: geometry collision mesh filename=package://kinova_description/meshes/finger_proximal.dae; visual mesh filename=package://kinova_description/meshes/finger_proximal.dae
- link m1n6s300_link_finger_3: geometry collision mesh filename=package://kinova_description/meshes/finger_proximal.dae; visual mesh filename=package://kinova_description/meshes/finger_proximal.dae
